Commit message: megarover

File: potbot_description/urdf/megarover.urdf.xacro (robot description, xacro)
@@ -12,17 +12,17 @@
     <color rgba="0.2 0.2 0.2 1" />
   </material>
-  <link name="horizontal_laser_link">
+  <link name="laser">
     <visual>
-      <origin xyz="0 0 -0.08" />
+      <origin xyz="0 0 -0.035" />
       <geometry>
-        <cylinder length="0.05" radius="0.03" />
+        <cylinder length="0.07" radius="0.0175" />
       </geometry>
       <material name="gray" />
     </visual>
   </link>
-  <joint name="horizontal_laser_link_joint" type="fixed">
+  <joint name="laser_joint" type="fixed">
     <parent link="base_link" />
-    <child link="horizontal_laser_link" />
-    <origin xyz="1 0 0.5"/>
+    <child link="laser" />
+    <origin xyz="0.09 0 0.234"/>
   </joint>
 </robot>

Commit message: add camera

File: potbot_description/urdf/megarover.urdf.xacro (robot description, xacro)
@@ -26,3 +26,29 @@
     <origin xyz="0.09 0 0.234"/>
   </joint>
+  <joint name="camera_joint" type="fixed">
+    <origin xyz="0 0 0.3" rpy="0 0 0"/>
+    <parent link="base_link"/>
+    <child link="camera_link"/>
+  </joint>
+  <link name="camera_link">
+    <visual>
+      <origin xyz="0 0 0" rpy="0 0 0"/>
+      <geometry>
+        <box size="0.02 0.1 0.02"/>
+      </geometry>
+      <material name="gray" />
+    </visual>
+  </link>
+  <joint name="camera_rgb_joint" type="fixed">
+    <origin xyz="0.003 0.011 0.009" rpy="0 0 0"/>
+    <parent link="camera_link"/>
+    <child link="camera_rgb_frame"/>
+  </joint>
+  <link name="camera_rgb_frame"/>
+  <joint name="camera_rgb_optical_joint" type="fixed">
+    <origin xyz="0 0 0" rpy="-1.57 0 -1.57"/>
+    <parent link="camera_rgb_frame"/>
+    <child link="camera_rgb_optical_frame"/>
+  </joint>
+  <link name="camera_rgb_optical_frame"/>
 </robot>
