Commit message: add beedo model

File: potbot_description/urdf/beego2.gazebo.xacro (robot description, xacro)
@@ -19,21 +19,4 @@
     <mu2 value="1.0" />
   </gazebo>
-  <!-- <gazebo>
-    <plugin name="pan_motor_controller" filename="libgazebo_ros_joint_position.so">
-      <commandTopic>set_position</commandTopic>
-      <odometryTopic>odom</odometryTopic>
-      <odometryFrame>odom</odometryFrame>
-      <odometrySource>world</odometrySource>
-      <publishOdomTF>true</publishOdomTF>
-      <robotBaseFrame>base_footprint</robotBaseFrame>
-      <publishWheelTF>false</publishWheelTF>
-      <publishTf>true</publishTf>
-      <publishWheelJointState>true</publishWheelJointState>
-      <legacyMode>false</legacyMode>
-      <updateRate>30</updateRate>
-      <Joint>camera_joint</Joint>
-      <rosDebugLevel>na</rosDebugLevel>
-    </plugin>
-  </gazebo> -->
   <gazebo>
     <plugin name="megarover21_controller" filename="libgazebo_ros_diff_drive.so">
@@ -121,3 +104,10 @@
     </sensor>
   </gazebo>
+  <gazebo>
+    <plugin name="gazebo_ros_control" filename="libgazebo_ros_control.so">
+      <!-- <robotNamespace>/beego2</robotNamespace> -->
+      <robotSimType>gazebo_ros_control/DefaultRobotHWSim</robotSimType>
+      <legacyModeNS>true</legacyModeNS>
+    </plugin>
+  </gazebo>
 </robot>

File: potbot_description/urdf/beego2.urdf.xacro (robot description, xacro)
@@ -4,7 +4,7 @@
   <xacro:include filename="$(find turtlebot3_description)/urdf/common_properties.xacro"/>
   <xacro:include filename="$(find potbot_description)/urdf/beego2.gazebo.xacro"/>
-  <xacro:property name="wheel_radius" value="0.076"/>
-  <xacro:property name="wheel_length" value="0.03"/>
-  <xacro:property name="wheel_mass" value="0.823"/>
+  <xacro:property name="wheel_radius" value="0.03"/>
+  <xacro:property name="wheel_length" value="0.015"/>
+  <xacro:property name="wheel_mass" value="0.4"/>
   <link name="base_footprint"/>
   <joint name="base_joint" type="fixed">
@@ -15,43 +15,43 @@
   <link name="base_link">
     <visual>
-      <geometry>
-        <mesh filename="package://megarover_samples/meshes/dae/vmega_body.dae"/>
-      </geometry>
-    </visual>
-    <collision>
-      <geometry>
-        <mesh filename="package://megarover_samples/meshes/stl/vmega_body.stl"/>
-      </geometry>
-    </collision>
-    <inertial>
-      <origin xyz="-0.061 0 -0.002"/>
-      <mass value="13.754"/>
-      <inertia ixx="0.110655982" ixy="0" ixz="0"
-        iyy="0.20062619" iyz="0"
-        izz="0.269504336" />
-    </inertial>
+      <origin xyz="-0.08 0 0.1"/>
+      <geometry>
+        <box size="0.2 0.2 0.2"/>
+      </geometry>
+    </visual>
+    <collision>
+      <origin xyz="-0.08 0.1"/>
+      <geometry>
+        <box size="0.2 0.2 0.2"/>
+      </geometry>
+    </collision>
+    <!-- <inertial>
+      <origin xyz="-0.08 0 0.1"/>
+      <mass value="5"/>
+      <inertia ixx="1" ixy="0" ixz="0" iyy="1" iyz="0" izz="1" />
+    </inertial> -->
   </link>
   <joint name="wheel_left_joint" type="continuous">
     <parent link="base_link"/>
     <child link="wheel_left_link"/>
-    <origin xyz="0 0.14199 0.074742"  rpy="0 0 ${M_PI}" />
+    <origin xyz="0 0.11 ${wheel_radius/2}"  rpy="0 0 ${M_PI}" />
     <axis xyz="0 -1 0"/>
   </joint>
   <link name="wheel_left_link">
     <visual>
-      <geometry>
-        <mesh filename="package://megarover_samples/meshes/dae/vmega_wheel.dae"/>
-      </geometry>
-    </visual>
-    <collision>
-      <origin xyz="0 0 0" rpy="${-M_PI/2} 0 0"/>
-      <geometry>
-        <cylinder radius="${wheel_radius}" length="${wheel_length}"/>
-      </geometry>
-    </collision>
-    <inertial>
-      <origin xyz="0 0 0" rpy="${-M_PI/2} 0 0"/>
-      <xacro:cylinder_inertial mass="${wheel_mass}"
-        radius="${wheel_radius}" length="${wheel_length}"/>
+      <origin xyz="0 0 0" rpy="${-M_PI/2} 0 0"/>
+      <geometry>
+        <cylinder radius="${wheel_radius}" length="${wheel_length}"/>
+      </geometry>
+    </visual>
+    <collision>
+      <origin xyz="0 0 0" rpy="${-M_PI/2} 0 0"/>
+      <geometry>
+        <cylinder radius="${wheel_radius}" length="${wheel_length}"/>
+      </geometry>
+    </collision>
+    <inertial>
+      <origin xyz="0 0 0" rpy="${-M_PI/2} 0 0"/>
+      <xacro:cylinder_inertial mass="${wheel_mass}" radius="${wheel_radius}" length="${wheel_length}"/>
     </inertial>
   </link>
@@ -59,23 +59,46 @@
     <parent link="base_link"/>
     <child link="wheel_right_link"/>
-    <origin xyz="0 -0.14199 0.074742"/>
+    <origin xyz="0 -0.11 ${wheel_radius/2}"/>
     <axis xyz="0 1 0"/>
   </joint>
   <link name="wheel_right_link">
     <visual>
-      <geometry>
-        <mesh filename="package://megarover_samples/meshes/dae/vmega_wheel.dae"/>
-      </geometry>
-    </visual>
-    <collision>
-      <origin xyz="0 0 0" rpy="${-M_PI/2} 0 0"/>
-      <geometry>
-        <cylinder radius="${wheel_radius}" length="${wheel_length}"/>
-      </geometry>
-    </collision>
-    <inertial>
-      <origin xyz="0 0 0" rpy="${-M_PI/2} 0 0"/>
-      <xacro:cylinder_inertial mass="${wheel_mass}"
-        radius="${wheel_radius}" length="${wheel_length}"/>
+      <origin xyz="0 0 0" rpy="${M_PI/2} 0 0"/>
+      <geometry>
+        <cylinder radius="${wheel_radius}" length="${wheel_length}"/>
+      </geometry>
+    </visual>
+    <collision>
+      <origin xyz="0 0 0" rpy="${M_PI/2} 0 0"/>
+      <geometry>
+        <cylinder radius="${wheel_radius}" length="${wheel_length}"/>
+      </geometry>
+    </collision>
+    <inertial>
+      <origin xyz="0 0 0" rpy="${M_PI/2} 0 0"/>
+      <xacro:cylinder_inertial mass="${wheel_mass}" radius="${wheel_radius}" length="${wheel_length}"/>
+    </inertial>
+  </link>
+  <joint name="caster_back_joint" type="fixed">
+    <parent link="base_link"/>
+    <child link="caster_back_link"/>
+    <origin xyz="-0.18 0 ${wheel_radius/2}" rpy="0 0 0"/>
+  </joint>
+  <link name="caster_back_link">
+    <visual>
+      <origin xyz="0 0 0" rpy="${-M_PI/2} 0 0"/>
+      <geometry>
+        <cylinder radius="${wheel_radius}" length="${wheel_length}"/>
+      </geometry>
+    </visual>
+    <collision>
+      <origin xyz="0 0 0" rpy="${-M_PI/2} 0 0"/>
+      <geometry>
+        <cylinder radius="${wheel_radius}" length="${wheel_length}"/>
+      </geometry>
+    </collision>
+    <inertial>
+      <origin xyz="0 0 0" rpy="${-M_PI/2} 0 0"/>
+      <xacro:cylinder_inertial mass="${wheel_mass}" radius="${wheel_radius}" length="${wheel_length}"/>
     </inertial>
   </link>
@@ -101,7 +124,69 @@
     </inertial>
   </link>
+  <joint name="pan_joint" type="revolute">
+    <axis xyz="0 0 1"/>
+    <origin xyz="0.06 0 0.455" rpy="0 0 0"/>
+    <limit lower="-1" upper="1" effort="100" velocity="100"/>
+    <parent link="base_link"/>
+    <child link="pan_link"/>
+  </joint>
+  <transmission name="pan_trans">
+    <type>transmission_interface/SimpleTransmission</type>
+    <joint name="pan_joint">
+      <hardwareInterface>hardware_interface/PositionJointInterface</hardwareInterface>
+    </joint>
+    <actuator name="pan_motor">
+       <hardwareInterface>hardware_interface/PositionJointInterface</hardwareInterface>
+       <mechanismReduction>1</mechanismReduction>
+    </actuator>
+  </transmission>
+  <link name="pan_link">
+    <visual>
+      <origin xyz="0 0 0" rpy="0 0 0"/>
+      <geometry>
+        <box size="0.01 0.01 0.01"/>
+      </geometry>
+      <material name="black" />
+    </visual>
+    <inertial>
+      <mass value="0.01"/>
+      <origin xyz="0 0 0" rpy="0 0 0"/>
+      <inertia ixx="1.0" ixy="0.0" ixz="0.0" iyy="1.0" iyz="0.0" izz="1.0"/>
+    </inertial>
+  </link>
+  <joint name="tilt_joint" type="revolute">
+    <axis xyz="0 1 0"/>
+    <origin xyz="0 -0.0825 0.015" rpy="0 0 0"/>
+    <limit lower="-1" upper="1" effort="100" velocity="100"/>
+    <parent link="pan_link"/>
+    <child link="tilt_link"/>
+  </joint>
+  <transmission name="tilt_trans">
+    <type>transmission_interface/SimpleTransmission</type>
+    <joint name="tilt_joint">
+      <hardwareInterface>hardware_interface/PositionJointInterface</hardwareInterface>
+    </joint>
+    <actuator name="tilt_motor">
+       <hardwareInterface>hardware_interface/PositionJointInterface</hardwareInterface>
+       <mechanismReduction>1</mechanismReduction>
+    </actuator>
+  </transmission>
+  <link name="tilt_link">
+    <visual>
+      <origin xyz="0 0 0" rpy="0 0 0"/>
+      <geometry>
+        <box size="0.01 0.01 0.01"/>
+      </geometry>
+      <material name="black" />
+    </visual>
+    <inertial>
+      <mass value="0.01"/>
+      <origin xyz="0 0 0" rpy="0 0 0"/>
+      <inertia ixx="1.0" ixy="0.0" ixz="0.0" iyy="1.0" iyz="0.0" izz="1.0"/>
+    </inertial>
+  </link>
   <joint name="camera_joint" type="fixed">
-    <origin xyz="0.06 0 0.455" rpy="0 0 0"/>
-    <parent link="base_link"/>
+    <origin xyz="0 0.0825 0" rpy="0 0 0"/>
+    <parent link="tilt_link"/>
     <child link="camera_link"/>
   </joint>
@@ -114,4 +199,15 @@
       <material name="gray" />
     </visual>
+    <collision>
+      <origin xyz="0 0 0" rpy="0 0 0"/>
+      <geometry>
+        <box size="0.03 0.165 0.03"/>
+      </geometry>
+    </collision>
+    <!-- <inertial>
+      <mass value="1.0"/>
+      <origin xyz="0 0 0" rpy="0 0 0"/>
+      <inertia ixx="1.0" ixy="0.0" ixz="0.0" iyy="1.0" iyz="0.0" izz="1.0"/>
+    </inertial> -->
   </link>
   <joint name="camera_rgb_joint" type="fixed">
@@ -127,13 +223,13 @@
   </joint>
   <link name="camera_rgb_optical_frame"/>
-  <transmission name="pan_motor_transmission">
+  <!-- <transmission name="pan_motor_transmission">
     <type>transmission_interface/SimpleTransmission</type>
     <joint name="camera_joint">
-      <hardwareInterface>PositionJointInterface</hardwareInterface>
+      <hardwareInterface>hardware_interface/PositionJointInterface</hardwareInterface>
     </joint>
     <actuator name="pan_motor">
-      <mechanicalReduction>30</mechanicalReduction>
-      <hardwareInterface>PositionJointInterface</hardwareInterface>
+      <mechanicalReduction>1</mechanicalReduction>
+      <hardwareInterface>hardware_interface/PositionJointInterface</hardwareInterface>
     </actuator>
-  </transmission>
+  </transmission> -->
 </robot>
