Commit message: desktop

File: potbot_description/urdf/beego2.gazebo.xacro (robot description, xacro)
@@ -5,4 +5,5 @@
   <xacro:arg name="imu_visual"    default="false"/>
   <gazebo reference="base_link">
+    <material>Gazebo/Grey</material>
     <selfCollide>false</selfCollide>
     <mu1 value="0.0" />
@@ -18,4 +19,16 @@
     <mu1 value="1.0" />
     <mu2 value="1.0" />
+  </gazebo>
+  <gazebo reference="caster_back_link">
+    <material>Gazebo/Black</material>
+  </gazebo>
+  <gazebo reference="camera_stay_link">
+    <material>Gazebo/Grey</material>
+  </gazebo>
+  <gazebo reference="pan_link">
+    <material>Gazebo/Black</material>
+  </gazebo>
+  <gazebo reference="tilt_link">
+    <material>Gazebo/Black</material>
   </gazebo>
   <gazebo>
@@ -44,5 +57,5 @@
     <sensor type="ray" name="urg_lrf_sensor">
       <pose>0 0 0 0 0 0</pose>
-      <visualize>true</visualize>
+      <visualize>$(arg laser_visual)</visualize>
       <update_rate>40</update_rate>
       <ray>
@@ -72,33 +85,48 @@
     </sensor>
   </gazebo>
-  <gazebo reference="camera_rgb_frame">
+  <gazebo reference="stereo_camera_frame">
     <sensor type="camera" name="Pi Camera">
       <always_on>true</always_on>
-      <visualize>true</visualize>
+      <visualize>$(arg camera_visual)</visualize>
+    </sensor>
+  </gazebo>
+  <gazebo reference="stereo_camera_frame">
+    <sensor name="depth_camera" type="depth">
+      <update_rate>20</update_rate>
       <camera>
-          <horizontal_fov>1.085595</horizontal_fov>
-          <image>
-              <width>640</width>
-              <height>480</height>
-              <format>R8G8B8</format>
-          </image>
-          <clip>
-              <near>0.03</near>
-              <far>100</far>
-          </clip>
+        <horizontal_fov>1.047198</horizontal_fov>
+        <image>
+          <width>640</width>
+          <height>480</height>
+          <format>R8G8B8</format>
+        </image>
+        <clip>
+          <near>0.05</near>
+          <far>3</far>
+        </clip>
       </camera>
-      <plugin name="camera_controller" filename="libgazebo_ros_camera.so">
+      <plugin name="depth_camera_controller" filename="libgazebo_ros_openni_kinect.so">
+        <baseline>0.2</baseline>
         <alwaysOn>true</alwaysOn>
-        <updateRate>30.0</updateRate>
-        <cameraName>camera</cameraName>
-        <frameName>camera_rgb_optical_frame</frameName>
-        <imageTopicName>rgb/image_raw</imageTopicName>
-        <cameraInfoTopicName>rgb/camera_info</cameraInfoTopicName>
-        <hackBaseline>0.07</hackBaseline>
-        <distortionK1>0.0</distortionK1>
-        <distortionK2>0.0</distortionK2>
-        <distortionK3>0.0</distortionK3>
-        <distortionT1>0.0</distortionT1>
-        <distortionT2>0.0</distortionT2>
+        <updateRate>1.0</updateRate>
+        <cameraName>realsense</cameraName>
+        <imageTopicName>color/image_raw</imageTopicName>
+        <cameraInfoTopicName>color/camera_info</cameraInfoTopicName>
+        <depthImageTopicName>depth/image_raw</depthImageTopicName>
+        <depthImageInfoTopicName>depth/camera_info</depthImageInfoTopicName>
+        <pointCloudTopicName>depth/points</pointCloudTopicName>
+        <frameName>stereo_camera_optical_frame</frameName>
+        <pointCloudCutoff>0.5</pointCloudCutoff>
+        <pointCloudCutoffMax>3.0</pointCloudCutoffMax>
+        <distortionK1>0.00000001</distortionK1>
+        <distortionK2>0.00000001</distortionK2>
+        <distortionK3>0.00000001</distortionK3>
+        <distortionT1>0.00000001</distortionT1>
+        <distortionT2>0.00000001</distortionT2>
+        <CxPrime>0</CxPrime>
+        <Cx>0</Cx>
+        <Cy>0</Cy>
+        <focalLength>0</focalLength>
+        <hackBaseline>0</hackBaseline>
       </plugin>
     </sensor>

File: potbot_description/urdf/beego2.urdf.xacro (robot description, xacro)
@@ -19,4 +19,5 @@
         <box size="0.2 0.2 0.2"/>
       </geometry>
+      <material name="grey" />
     </visual>
     <collision>
@@ -26,9 +27,8 @@
       </geometry>
     </collision>
-    <!-- <inertial>
-      <origin xyz="-0.08 0 0.1"/>
-      <mass value="5"/>
-      <inertia ixx="1" ixy="0" ixz="0" iyy="1" iyz="0" izz="1" />
-    </inertial> -->
+    <inertial>
+      <origin xyz="0 0 0"/>
+      <xacro:box_inertial mass="5" height="0.2" width="0.2" depth="0.2"/>
+    </inertial>
   </link>
   <joint name="wheel_left_joint" type="continuous">
@@ -44,4 +44,5 @@
         <cylinder radius="${wheel_radius}" length="${wheel_length}"/>
       </geometry>
+      <material name="white" />
     </visual>
     <collision>
@@ -68,4 +69,5 @@
         <cylinder radius="${wheel_radius}" length="${wheel_length}"/>
       </geometry>
+      <material name="white" />
     </visual>
     <collision>
@@ -91,14 +93,15 @@
         <cylinder radius="${wheel_radius}" length="${wheel_length}"/>
       </geometry>
-    </visual>
-    <collision>
-      <origin xyz="0 0 0" rpy="${-M_PI/2} 0 0"/>
-      <geometry>
-        <cylinder radius="${wheel_radius}" length="${wheel_length}"/>
-      </geometry>
-    </collision>
-    <inertial>
-      <origin xyz="0 0 0" rpy="${-M_PI/2} 0 0"/>
-      <xacro:cylinder_inertial mass="${wheel_mass}" radius="${wheel_radius}" length="${wheel_length}"/>
+      <material name="black" />
+    </visual>
+    <collision>
+      <origin xyz="0 0 0" rpy="${-M_PI/2} 0 0"/>
+      <geometry>
+        <cylinder radius="${wheel_radius}" length="${wheel_length}"/>
+      </geometry>
+    </collision>
+    <inertial>
+      <origin xyz="0 0 0" rpy="${-M_PI/2} 0 0"/>
+      <xacro:cylinder_inertial mass="${wheel_mass*5}" radius="${wheel_radius}" length="${wheel_length}"/>
     </inertial>
   </link>
@@ -124,9 +127,33 @@
     </inertial>
   </link>
+  <joint name="camera_stay_joint" type="fixed">
+    <origin xyz="0.06 0 0.2275" rpy="0 0 0"/>
+    <parent link="base_link"/>
+    <child link="camera_stay_link"/>
+  </joint>
+  <link name="camera_stay_link">
+    <visual>
+      <origin xyz="0 0 0" rpy="0 0 0"/>
+      <geometry>
+        <box size="0.02 0.02 0.455"/>
+      </geometry>
+      <material name="grey" />
+    </visual>
+    <collision>
+      <origin xyz="0 0 0" rpy="0 0 0"/>
+      <geometry>
+        <box size="0.02 0.02 0.455"/>
+      </geometry>
+    </collision>
+    <inertial>
+      <origin xyz="0 0 0"/>
+      <xacro:box_inertial mass="0.5" height="0.455" width="0.02" depth="0.02"/>
+    </inertial>
+  </link>
   <joint name="pan_joint" type="revolute">
     <axis xyz="0 0 1"/>
-    <origin xyz="0.06 0 0.455" rpy="0 0 0"/>
+    <origin xyz="0 0 0.2375" rpy="0 0 0"/>
     <limit lower="-1" upper="1" effort="100" velocity="100"/>
-    <parent link="base_link"/>
+    <parent link="camera_stay_link"/>
     <child link="pan_link"/>
   </joint>
@@ -150,7 +177,6 @@
     </visual>
     <inertial>
-      <mass value="0.01"/>
-      <origin xyz="0 0 0" rpy="0 0 0"/>
-      <inertia ixx="1.0" ixy="0.0" ixz="0.0" iyy="1.0" iyz="0.0" izz="1.0"/>
+      <origin xyz="0 0 0"/>
+      <xacro:box_inertial mass="0.1" height="0.01" width="0.01" depth="0.01"/>
     </inertial>
   </link>
@@ -181,7 +207,6 @@
     </visual>
     <inertial>
-      <mass value="0.01"/>
-      <origin xyz="0 0 0" rpy="0 0 0"/>
-      <inertia ixx="1.0" ixy="0.0" ixz="0.0" iyy="1.0" iyz="0.0" izz="1.0"/>
+      <origin xyz="0 0 0"/>
+      <xacro:box_inertial mass="0.1" height="0.01" width="0.01" depth="0.01"/>
     </inertial>
   </link>
@@ -197,5 +222,5 @@
         <box size="0.03 0.165 0.03"/>
       </geometry>
-      <material name="gray" />
+      <material name="white" />
     </visual>
     <collision>
@@ -205,31 +230,16 @@
       </geometry>
     </collision>
-    <!-- <inertial>
-      <mass value="1.0"/>
-      <origin xyz="0 0 0" rpy="0 0 0"/>
-      <inertia ixx="1.0" ixy="0.0" ixz="0.0" iyy="1.0" iyz="0.0" izz="1.0"/>
-    </inertial> -->
-  </link>
-  <joint name="camera_rgb_joint" type="fixed">
+  </link>
+  <joint name="stereo_camera_joint" type="fixed">
     <origin xyz="0 0 0" rpy="0 0 0"/>
     <parent link="camera_link"/>
-    <child link="camera_rgb_frame"/>
-  </joint>
-  <link name="camera_rgb_frame"/>
-  <joint name="camera_rgb_optical_joint" type="fixed">
+    <child link="stereo_camera_frame"/>
+  </joint>
+  <link name="stereo_camera_frame"/>
+  <joint name="stereo_camera_optical_joint" type="fixed">
     <origin xyz="0 0 0" rpy="-1.57 0 -1.57"/>
-    <parent link="camera_rgb_frame"/>
-    <child link="camera_rgb_optical_frame"/>
-  </joint>
-  <link name="camera_rgb_optical_frame"/>
-  <!-- <transmission name="pan_motor_transmission">
-    <type>transmission_interface/SimpleTransmission</type>
-    <joint name="camera_joint">
-      <hardwareInterface>hardware_interface/PositionJointInterface</hardwareInterface>
-    </joint>
-    <actuator name="pan_motor">
-      <mechanicalReduction>1</mechanicalReduction>
-      <hardwareInterface>hardware_interface/PositionJointInterface</hardwareInterface>
-    </actuator>
-  </transmission> -->
+    <parent link="stereo_camera_frame"/>
+    <child link="stereo_camera_optical_frame"/>
+  </joint>
+  <link name="stereo_camera_optical_frame"/>
 </robot>

File: potbot_description/urdf/megarover21.gazebo.xacro (robot description, xacro)
@@ -18,4 +18,7 @@
     <mu1 value="1.0" />
     <mu2 value="1.0" />
+  </gazebo>
+  <gazebo reference="camera_stay_link">
+    <material>Gazebo/Grey</material>
   </gazebo>
   <gazebo>
@@ -44,5 +47,5 @@
     <sensor type="ray" name="urg_lrf_sensor">
       <pose>0 0 0 0 0 0</pose>
-      <visualize>true</visualize>
+      <visualize>$(arg laser_visual)</visualize>
       <update_rate>40</update_rate>
       <ray>
@@ -72,9 +75,9 @@
     </sensor>
   </gazebo>
-  <gazebo reference="camera_rgb_frame">
+  <gazebo reference="stereo_camera_frame">
     <sensor type="camera" name="Pi Camera">
       <always_on>true</always_on>
-      <visualize>true</visualize>
-      <camera>
+      <visualize>$(arg camera_visual)</visualize>
+      <!-- <camera>
           <horizontal_fov>1.085595</horizontal_fov>
           <image>
@@ -92,5 +95,5 @@
         <updateRate>30.0</updateRate>
         <cameraName>camera</cameraName>
-        <frameName>camera_rgb_optical_frame</frameName>
+        <frameName>stereo_camera_optical_frame</frameName>
         <imageTopicName>rgb/image_raw</imageTopicName>
         <cameraInfoTopicName>rgb/camera_info</cameraInfoTopicName>
@@ -101,6 +104,102 @@
         <distortionT1>0.0</distortionT1>
         <distortionT2>0.0</distortionT2>
+      </plugin> -->
+    </sensor>
+  </gazebo>
+  <!-- <gazebo reference="stereo_camera_frame">
+    <sensor type="multicamera" name="stereo_camera">
+      <always_on>true</always_on>
+      <update_rate>30.0</update_rate>
+      <camera name="left">
+        <horizontal_fov>1.3962634</horizontal_fov>
+        <image>
+          <width>800</width>
+          <height>800</height>
+          <format>R8G8B8</format>
+        </image>
+        <clip>
+          <near>0.02</near>
+          <far>300</far>
+        </clip>
+        <noise>
+          <type>gaussian</type>
+          <mean>0.0</mean>
+          <stddev>0.007</stddev>
+        </noise>
+      </camera>
+      <camera name="right">
+        <pose>0 -0.07 0 0 0 0</pose>
+        <horizontal_fov>1.3962634</horizontal_fov>
+        <image>
+          <width>800</width>
+          <height>800</height>
+          <format>R8G8B8</format>
+        </image>
+        <clip>
+          <near>0.02</near>
+          <far>300</far>
+        </clip>
+        <noise>
+          <type>gaussian</type>
+          <mean>0.0</mean>
+          <stddev>0.007</stddev>
+        </noise>
+      </camera>
+      <plugin name="stereo_camera_controller" filename="libgazebo_ros_multicamera.so">
+        <alwaysOn>true</alwaysOn>
+        <updateRate>0.0</updateRate>
+        <cameraName>mynteye</cameraName>
+        <imageTopicName>image_raw</imageTopicName>
+        <cameraInfoTopicName>camera_info</cameraInfoTopicName>
+        <frameName>stereo_camera_optical_frame</frameName>
+        <hackBaseline>0.07</hackBaseline>
+        <distortionK1>0.0</distortionK1>
+        <distortionK2>0.0</distortionK2>
+        <distortionK3>0.0</distortionK3>
+        <distortionT1>0.0</distortionT1>
+        <distortionT2>0.0</distortionT2>
       </plugin>
     </sensor>
+  </gazebo> -->
+  <gazebo reference="stereo_camera_frame">
+    <sensor name="depth_camera" type="depth">
+      <update_rate>20</update_rate>
+      <camera>
+        <horizontal_fov>1.047198</horizontal_fov>
+        <image>
+          <width>640</width>
+          <height>480</height>
+          <format>R8G8B8</format>
+        </image>
+        <clip>
+          <near>0.05</near>
+          <far>3</far>
+        </clip>
+      </camera>
+      <plugin name="depth_camera_controller" filename="libgazebo_ros_openni_kinect.so">
+        <baseline>0.2</baseline>
+        <alwaysOn>true</alwaysOn>
+        <updateRate>1.0</updateRate>
+        <cameraName>realsense</cameraName>
+        <imageTopicName>color/image_raw</imageTopicName>
+        <cameraInfoTopicName>color/camera_info</cameraInfoTopicName>
+        <depthImageTopicName>depth/image_raw</depthImageTopicName>
+        <depthImageInfoTopicName>depth/camera_info</depthImageInfoTopicName>
+        <pointCloudTopicName>depth/points</pointCloudTopicName>
+        <frameName>stereo_camera_optical_frame</frameName>
+        <pointCloudCutoff>0.5</pointCloudCutoff>
+        <pointCloudCutoffMax>3.0</pointCloudCutoffMax>
+        <distortionK1>0.00000001</distortionK1>
+        <distortionK2>0.00000001</distortionK2>
+        <distortionK3>0.00000001</distortionK3>
+        <distortionT1>0.00000001</distortionT1>
+        <distortionT2>0.00000001</distortionT2>
+        <CxPrime>0</CxPrime>
+        <Cx>0</Cx>
+        <Cy>0</Cy>
+        <focalLength>0</focalLength>
+        <hackBaseline>0</hackBaseline>
+      </plugin>
+    </sensor>
   </gazebo>
 </robot>

File: potbot_description/urdf/megarover21.urdf.xacro (robot description, xacro)
@@ -84,5 +84,5 @@
     <child link="base_scan" />
     <!-- <origin xyz="0.09 0 0.234"/> -->
-    <origin xyz="0.09 0 0.223" rpy="${M_PI} 0 0"/>
+    <origin xyz="0.09 0 0.223" rpy="0 0 0"/>
   </joint>
   <!-- <link name="base_scan">
@@ -92,9 +92,10 @@
         <cylinder length="0.07" radius="0.0175" />
       </geometry>
-      <material name="gray" />
+      <material name="grey" />
     </visual>
   </link> -->
   <link name="base_scan">
     <visual>
+      <origin xyz="0 0 0" rpy="${M_PI} 0 0"/>
       <geometry>
         <mesh filename="package://megarover_samples/meshes/dae/lrf.dae"/>
@@ -111,7 +112,27 @@
     </inertial>
   </link>
+  <joint name="camera_stay_joint" type="fixed">
+    <origin xyz="0.06 0 0.2275" rpy="0 0 0"/>
+    <parent link="base_link"/>
+    <child link="camera_stay_link"/>
+  </joint>
+  <link name="camera_stay_link">
+    <visual>
+      <origin xyz="0 0 0" rpy="0 0 0"/>
+      <geometry>
+        <box size="0.02 0.02 0.455"/>
+      </geometry>
+      <material name="grey" />
+    </visual>
+    <collision>
+      <origin xyz="0 0 0" rpy="0 0 0"/>
+      <geometry>
+        <box size="0.02 0.02 0.455"/>
+      </geometry>
+    </collision>
+  </link>
   <joint name="camera_joint" type="fixed">
-    <origin xyz="0.06 0 0.455" rpy="0 0 0"/>
-    <parent link="base_link"/>
+    <origin xyz="0 0 0.2275" rpy="0 0 0"/>
+    <parent link="camera_stay_link"/>
     <child link="camera_link"/>
   </joint>
@@ -122,18 +143,18 @@
         <box size="0.03 0.165 0.03"/>
       </geometry>
-      <material name="gray" />
+      <material name="white" />
     </visual>
   </link>
-  <joint name="camera_rgb_joint" type="fixed">
+  <joint name="stereo_camera_joint" type="fixed">
     <origin xyz="0 0 0" rpy="0 0 0"/>
     <parent link="camera_link"/>
-    <child link="camera_rgb_frame"/>
+    <child link="stereo_camera_frame"/>
   </joint>
-  <link name="camera_rgb_frame"/>
-  <joint name="camera_rgb_optical_joint" type="fixed">
+  <link name="stereo_camera_frame"/>
+  <joint name="stereo_camera_optical_joint" type="fixed">
     <origin xyz="0 0 0" rpy="-1.57 0 -1.57"/>
-    <parent link="camera_rgb_frame"/>
-    <child link="camera_rgb_optical_frame"/>
+    <parent link="stereo_camera_frame"/>
+    <child link="stereo_camera_optical_frame"/>
   </joint>
-  <link name="camera_rgb_optical_frame"/>
+  <link name="stereo_camera_optical_frame"/>
 </robot>

Commit message: desktop

File: potbot_description/urdf/beego2.gazebo.xacro (robot description, xacro)
@@ -97,5 +97,5 @@
         <horizontal_fov>1.047198</horizontal_fov>
         <image>
-          <width>640</width>
+          <width>752</width>
           <height>480</height>
           <format>R8G8B8</format>

File: potbot_description/urdf/beego2.urdf.xacro (robot description, xacro)
@@ -154,5 +154,5 @@
     <axis xyz="0 0 1"/>
     <origin xyz="0 0 0.2375" rpy="0 0 0"/>
-    <limit lower="-1" upper="1" effort="100" velocity="100"/>
+    <limit lower="-0.87" upper="0.87" effort="100" velocity="100"/>
     <parent link="camera_stay_link"/>
     <child link="pan_link"/>
@@ -184,5 +184,5 @@
     <axis xyz="0 1 0"/>
     <origin xyz="0 -0.0825 0.015" rpy="0 0 0"/>
-    <limit lower="-1" upper="1" effort="100" velocity="100"/>
+    <limit lower="-0.87" upper="0.87" effort="100" velocity="100"/>
     <parent link="pan_link"/>
     <child link="tilt_link"/>
