Commit message: ros-pc

File: potbot_description/urdf/beego2.gazebo.xacro (robot description, xacro)
@@ -85,5 +85,5 @@
     </sensor>
   </gazebo>
-  <gazebo reference="stereo_camera_frame">
+  <gazebo reference="left_camera_frame">
     <sensor type="camera" name="Pi Camera">
       <always_on>true</always_on>
@@ -91,5 +91,5 @@
     </sensor>
   </gazebo>
-  <gazebo reference="stereo_camera_frame">
+  <gazebo reference="left_camera_frame">
     <sensor name="depth_camera" type="depth">
       <update_rate>20</update_rate>
@@ -116,5 +116,5 @@
         <depthImageInfoTopicName>depth/camera_info</depthImageInfoTopicName>
         <pointCloudTopicName>depth/points</pointCloudTopicName>
-        <frameName>stereo_camera_optical_frame</frameName>
+        <frameName>left_camera_optical_frame</frameName>
         <pointCloudCutoff>0.5</pointCloudCutoff>
         <pointCloudCutoffMax>3.0</pointCloudCutoffMax>

File: potbot_description/urdf/beego2.urdf.xacro (robot description, xacro)
@@ -28,5 +28,5 @@
     </collision>
     <inertial>
-      <origin xyz="0 0 0"/>
+      <origin xyz="0 0 0" rpy="0 0 0"/>
       <xacro:box_inertial mass="5" height="0.2" width="0.2" depth="0.23"/>
     </inertial>
@@ -109,8 +109,9 @@
     <parent link="base_link" />
     <child link="base_scan" />
-    <origin xyz="0.1 0 0.18" rpy="${M_PI} 0 0"/>
+    <origin xyz="0.1 0 0.18" rpy="0 0 0"/>
   </joint>
   <link name="base_scan">
     <visual>
+      <origin xyz="0 0 0" rpy="${M_PI} 0 0"/>
       <geometry>
         <mesh filename="package://megarover_samples/meshes/dae/lrf.dae"/>
@@ -118,4 +119,5 @@
     </visual>
     <collision>
+      <origin xyz="0 0 0" rpy="${M_PI} 0 0"/>
       <geometry>
         <mesh filename="package://megarover_samples/meshes/stl/lrf.stl"/>
@@ -231,15 +233,27 @@
     </collision>
   </link>
-  <joint name="stereo_camera_joint" type="fixed">
-    <origin xyz="0 0 0" rpy="0 0 0"/>
+  <joint name="left_camera_joint" type="fixed">
+    <origin xyz="0 0.06 0" rpy="0 0 0"/>
     <parent link="camera_link"/>
-    <child link="stereo_camera_frame"/>
-  </joint>
-  <link name="stereo_camera_frame"/>
-  <joint name="stereo_camera_optical_joint" type="fixed">
+    <child link="left_camera_frame"/>
+  </joint>
+  <link name="left_camera_frame"/>
+  <joint name="left_camera_optical_joint" type="fixed">
     <origin xyz="0 0 0" rpy="-1.57 0 -1.57"/>
-    <parent link="stereo_camera_frame"/>
-    <child link="stereo_camera_optical_frame"/>
-  </joint>
-  <link name="stereo_camera_optical_frame"/>
+    <parent link="left_camera_frame"/>
+    <child link="left_camera_optical_frame"/>
+  </joint>
+  <link name="left_camera_optical_frame"/>
+  <joint name="right_camera_joint" type="fixed">
+    <origin xyz="0 -0.06 0" rpy="0 0 0"/>
+    <parent link="camera_link"/>
+    <child link="right_camera_frame"/>
+  </joint>
+  <link name="right_camera_frame"/>
+  <joint name="right_camera_optical_joint" type="fixed">
+    <origin xyz="0 0 0" rpy="-1.57 0 -1.57"/>
+    <parent link="right_camera_frame"/>
+    <child link="right_camera_optical_frame"/>
+  </joint>
+  <link name="right_camera_optical_frame"/>
 </robot>

File: potbot_description/urdf/megarover21.gazebo.xacro (robot description, xacro)
@@ -75,5 +75,5 @@
     </sensor>
   </gazebo>
-  <gazebo reference="stereo_camera_frame">
+  <gazebo reference="left_camera_frame">
     <sensor type="camera" name="Pi Camera">
       <always_on>true</always_on>
@@ -95,5 +95,5 @@
         <updateRate>30.0</updateRate>
         <cameraName>camera</cameraName>
-        <frameName>stereo_camera_optical_frame</frameName>
+        <frameName>left_camera_optical_frame</frameName>
         <imageTopicName>rgb/image_raw</imageTopicName>
         <cameraInfoTopicName>rgb/camera_info</cameraInfoTopicName>
@@ -107,6 +107,6 @@
     </sensor>
   </gazebo>
-  <!-- <gazebo reference="stereo_camera_frame">
-    <sensor type="multicamera" name="stereo_camera">
+  <!-- <gazebo reference="left_camera_frame">
+    <sensor type="multicamera" name="left_camera">
       <always_on>true</always_on>
       <update_rate>30.0</update_rate>
@@ -146,5 +146,5 @@
         </noise>
       </camera>
-      <plugin name="stereo_camera_controller" filename="libgazebo_ros_multicamera.so">
+      <plugin name="left_camera_controller" filename="libgazebo_ros_multicamera.so">
         <alwaysOn>true</alwaysOn>
         <updateRate>0.0</updateRate>
@@ -152,5 +152,5 @@
         <imageTopicName>image_raw</imageTopicName>
         <cameraInfoTopicName>camera_info</cameraInfoTopicName>
-        <frameName>stereo_camera_optical_frame</frameName>
+        <frameName>left_camera_optical_frame</frameName>
         <hackBaseline>0.07</hackBaseline>
         <distortionK1>0.0</distortionK1>
@@ -162,5 +162,5 @@
     </sensor>
   </gazebo> -->
-  <gazebo reference="stereo_camera_frame">
+  <gazebo reference="left_camera_frame">
     <sensor name="depth_camera" type="depth">
       <update_rate>20</update_rate>
@@ -187,5 +187,5 @@
         <depthImageInfoTopicName>depth/camera_info</depthImageInfoTopicName>
         <pointCloudTopicName>depth/points</pointCloudTopicName>
-        <frameName>stereo_camera_optical_frame</frameName>
+        <frameName>left_camera_optical_frame</frameName>
         <pointCloudCutoff>0.5</pointCloudCutoff>
         <pointCloudCutoffMax>3.0</pointCloudCutoffMax>

File: potbot_description/urdf/megarover21.urdf.xacro (robot description, xacro)
@@ -103,4 +103,5 @@
     </visual>
     <collision>
+      <origin xyz="0 0 0" rpy="${M_PI} 0 0"/>
       <geometry>
         <mesh filename="package://megarover_samples/meshes/stl/lrf.stl"/>
@@ -113,5 +114,5 @@
   </link>
   <joint name="camera_stay_joint" type="fixed">
-    <origin xyz="0.06 0 0.2275" rpy="0 0 0"/>
+    <origin xyz="0.06 0 0.305" rpy="0 0 0"/>
     <parent link="base_link"/>
     <child link="camera_stay_link"/>
@@ -121,5 +122,5 @@
       <origin xyz="0 0 0" rpy="0 0 0"/>
       <geometry>
-        <box size="0.02 0.02 0.455"/>
+        <box size="0.02 0.02 0.3"/>
       </geometry>
       <material name="grey" />
@@ -128,10 +129,10 @@
       <origin xyz="0 0 0" rpy="0 0 0"/>
       <geometry>
-        <box size="0.02 0.02 0.455"/>
+        <box size="0.02 0.02 0.3"/>
       </geometry>
     </collision>
   </link>
   <joint name="camera_joint" type="fixed">
-    <origin xyz="0 0 0.2275" rpy="0 0 0"/>
+    <origin xyz="0 0 0.15" rpy="0 0 0"/>
     <parent link="camera_stay_link"/>
     <child link="camera_link"/>
@@ -146,15 +147,27 @@
     </visual>
   </link>
-  <joint name="stereo_camera_joint" type="fixed">
-    <origin xyz="0 0 0" rpy="0 0 0"/>
+  <joint name="left_camera_joint" type="fixed">
+    <origin xyz="0 0.06 0" rpy="0 0 0"/>
     <parent link="camera_link"/>
-    <child link="stereo_camera_frame"/>
+    <child link="left_camera_frame"/>
   </joint>
-  <link name="stereo_camera_frame"/>
-  <joint name="stereo_camera_optical_joint" type="fixed">
+  <link name="left_camera_frame"/>
+  <joint name="left_camera_optical_joint" type="fixed">
     <origin xyz="0 0 0" rpy="-1.57 0 -1.57"/>
-    <parent link="stereo_camera_frame"/>
-    <child link="stereo_camera_optical_frame"/>
+    <parent link="left_camera_frame"/>
+    <child link="left_camera_optical_frame"/>
   </joint>
-  <link name="stereo_camera_optical_frame"/>
+  <link name="left_camera_optical_frame"/>
+  <joint name="right_camera_joint" type="fixed">
+    <origin xyz="0 -0.06 0" rpy="0 0 0"/>
+    <parent link="camera_link"/>
+    <child link="right_camera_frame"/>
+  </joint>
+  <link name="right_camera_frame"/>
+  <joint name="right_camera_optical_joint" type="fixed">
+    <origin xyz="0 0 0" rpy="-1.57 0 -1.57"/>
+    <parent link="right_camera_frame"/>
+    <child link="right_camera_optical_frame"/>
+  </joint>
+  <link name="right_camera_optical_frame"/>
 </robot>
