Commit message: desktop

File: potbot_description/urdf/r2d2.urdf.xacro (robot description, xacro)
@@ -1,5 +1,5 @@
 <?xml version="1.0" ?>
-<robot name="r2d2" xmlns:xacro="http://ros.org/wiki/xacro">
-<xacro:include filename="$(find megarover_samples)/urdf/common.xacro"/>
+  <robot name="r2d2" xmlns:xacro="http://ros.org/wiki/xacro">
+  <xacro:include filename="$(find megarover_samples)/urdf/common.xacro"/>
   <link name="base_footprint"/>
   <joint name="base_joint" type="fixed">
@@ -12,11 +12,12 @@
       <origin xyz="0 0 0" rpy="0 0 1.57"/>
       <geometry>
-        <mesh filename="/home/ros/r2d2-flat-on-plate-1.stl" scale="0.01 0.01 0.01"/>
+        <mesh filename="$(env HOME)/gazebo/r2d2-flat-on-plate-1.stl" scale="0.01 0.01 0.01"/>
       </geometry>
+      <material name="blue" />
     </visual>
     <collision>
       <origin xyz="0 0 0" rpy="0 0 1.57"/>
       <geometry>
-        <mesh filename="/home/ros/r2d2-flat-on-plate-1.stl" scale="0.01 0.01 0.01"/>
+        <mesh filename="$(env HOME)/gazebo/r2d2-flat-on-plate-1.stl" scale="0.01 0.01 0.01"/>
       </geometry>
     </collision>
