Commit message: ros-pc

File: potbot_description/urdf/megarover21.gazebo.xacro (robot description, xacro)
@@ -75,4 +75,14 @@
     </sensor>
   </gazebo>
+  <gazebo>
+    <plugin name="imu_plugin" filename="libgazebo_ros_imu.so">
+      <alwaysOn>true</alwaysOn>
+      <bodyName>imu_link</bodyName>
+      <topicName>imu</topicName>
+      <serviceName>imu_service</serviceName>
+      <gaussianNoise>0.0</gaussianNoise>
+      <updateRate>20.0</updateRate>
+    </plugin>
+  </gazebo>
   <gazebo reference="left_camera_frame">
     <sensor type="camera" name="Pi Camera">

File: potbot_description/urdf/megarover21.urdf.xacro (robot description, xacro)
@@ -147,4 +147,10 @@
     </visual>
   </link>
+  <joint name="imu_joint" type="fixed">
+    <parent link="camera_link"/>
+    <child link="imu_link"/>
+    <origin xyz="0 0 0" rpy="0 0 0"/>
+  </joint>
+  <link name="imu_link"/>
   <joint name="left_camera_joint" type="fixed">
     <origin xyz="0 0.06 0" rpy="0 0 0"/>
