Commit message: desktop

File: potbot_description/urdf/lumine.urdf.xacro (robot description, xacro)
@@ -12,5 +12,5 @@
       <origin xyz="0 0 0" rpy="0 0 0"/>
       <geometry>
-        <mesh filename="$(env HOME)/gazebo/BB-8.stl" scale="0.0025 0.0025 0.0025"/>
+        <mesh filename="$(env HOME)/gazebo/lumine.stl" scale="0.0025 0.0025 0.0025"/>
       </geometry>
       <material name="grey" />
@@ -19,5 +19,5 @@
       <origin xyz="0 0 0" rpy="0 0 0"/>
       <geometry>
-        <mesh filename="$(env HOME)/gazebo/BB-8.stl" scale="0.0025 0.0025 0.0025"/>
+        <mesh filename="$(env HOME)/gazebo/lumine.stl" scale="0.0025 0.0025 0.0025"/>
       </geometry>
     </collision>
