Commit message: ros-pc

File: potbot_description/urdf/beego2.urdf.xacro (robot description, xacro)
@@ -1,7 +1,7 @@
 <?xml version="1.0" ?>
-<robot name="turtlebot3_waffle_pi" xmlns:xacro="http://ros.org/wiki/xacro">
+<robot name="beego2" xmlns:xacro="http://ros.org/wiki/xacro">
   <xacro:include filename="$(find megarover_samples)/urdf/common.xacro"/>
   <xacro:include filename="$(find turtlebot3_description)/urdf/common_properties.xacro"/>
-  <xacro:include filename="$(find potbot_description)/urdf/megarover_3.gazebo.xacro"/>
+  <xacro:include filename="$(find potbot_description)/urdf/beego2.gazebo.xacro"/>
   <xacro:property name="wheel_radius" value="0.076"/>
   <xacro:property name="wheel_length" value="0.03"/>
@@ -83,16 +83,6 @@
     <parent link="base_link" />
     <child link="base_scan" />
-    <!-- <origin xyz="0.09 0 0.234"/> -->
     <origin xyz="0.09 0 0.223" rpy="${M_PI} 0 0"/>
   </joint>
-  <!-- <link name="base_scan">
-    <visual>
-      <origin xyz="0 0 -0.035" />
-      <geometry>
-        <cylinder length="0.07" radius="0.0175" />
-      </geometry>
-      <material name="gray" />
-    </visual>
-  </link> -->
   <link name="base_scan">
     <visual>
@@ -112,5 +102,5 @@
   </link>
   <joint name="camera_joint" type="fixed">
-    <origin xyz="0 0 0.3" rpy="0 0 0"/>
+    <origin xyz="0.06 0 0.455" rpy="0 0 0"/>
     <parent link="base_link"/>
     <child link="camera_link"/>
@@ -120,5 +110,5 @@
       <origin xyz="0 0 0" rpy="0 0 0"/>
       <geometry>
-        <box size="0.02 0.1 0.02"/>
+        <box size="0.03 0.165 0.03"/>
       </geometry>
       <material name="gray" />
@@ -126,5 +116,5 @@
   </link>
   <joint name="camera_rgb_joint" type="fixed">
-    <origin xyz="0.003 0.011 0.009" rpy="0 0 0"/>
+    <origin xyz="0 0 0" rpy="0 0 0"/>
     <parent link="camera_link"/>
     <child link="camera_rgb_frame"/>
@@ -137,28 +127,13 @@
   </joint>
   <link name="camera_rgb_optical_frame"/>
-  <joint name="camera_joint" type="fixed">
-    <origin xyz="0.073 -0.011 0.084" rpy="0 0 0"/>
-    <parent link="base_link"/>
-    <child link="camera_link"/>
-  </joint>
-  <link name="camera_link">
-    <collision>
-      <origin xyz="0.005 0.011 0.013" rpy="0 0 0"/>
-      <geometry>
-        <box size="0.015 0.030 0.027"/>
-      </geometry>
-    </collision>
-  </link>
-  <joint name="camera_rgb_joint" type="fixed">
-    <origin xyz="0.003 0.011 0.009" rpy="0 0 0"/>
-    <parent link="camera_link"/>
-    <child link="camera_rgb_frame"/>
-  </joint>
-  <link name="camera_rgb_frame"/>
-  <joint name="camera_rgb_optical_joint" type="fixed">
-    <origin xyz="0 0 0" rpy="-1.57 0 -1.57"/>
-    <parent link="camera_rgb_frame"/>
-    <child link="camera_rgb_optical_frame"/>
-  </joint>
-  <link name="camera_rgb_optical_frame"/>
+  <transmission name="pan_motor_transmission">
+    <type>transmission_interface/SimpleTransmission</type>
+    <joint name="camera_joint">
+      <hardwareInterface>PositionJointInterface</hardwareInterface>
+    </joint>
+    <actuator name="pan_motor">
+      <mechanicalReduction>30</mechanicalReduction>
+      <hardwareInterface>PositionJointInterface</hardwareInterface>
+    </actuator>
+  </transmission>
 </robot>

File: potbot_description/urdf/megarover21.gazebo.xacro (robot description, xacro)
@@ -1,4 +1,4 @@
 <?xml version="1.0"?>
-<robot name="turtlebot3_waffle_pi_sim" xmlns:xacro="http://ros.org/wiki/xacro">
+<robot name="megarover21_sim" xmlns:xacro="http://ros.org/wiki/xacro">
   <xacro:arg name="laser_visual"  default="false"/>
   <xacro:arg name="camera_visual" default="false"/>
@@ -9,10 +9,10 @@
     <mu2 value="0.0" />
   </gazebo>
-  <gazebo reference="$wheel_left_link">
+  <gazebo reference="wheel_left_link">
     <selfCollide>false</selfCollide>
     <mu1 value="1.0" />
     <mu2 value="1.0" />
   </gazebo>
-  <gazebo reference="$wheel_right_link">
+  <gazebo reference="wheel_right_link">
     <selfCollide>false</selfCollide>
     <mu1 value="1.0" />
@@ -20,5 +20,5 @@
   </gazebo>
   <gazebo>
-    <plugin name="megarover2.1_controller" filename="libgazebo_ros_diff_drive.so">
+    <plugin name="megarover21_controller" filename="libgazebo_ros_diff_drive.so">
       <commandTopic>cmd_vel</commandTopic>
       <odometryTopic>odom</odometryTopic>
@@ -42,30 +42,29 @@
   </gazebo>
   <gazebo reference="base_scan">
-    <material>Gazebo/FlatBlack</material>
-    <sensor type="ray" name="lds_lfcd_sensor">
+    <sensor type="ray" name="urg_lrf_sensor">
       <pose>0 0 0 0 0 0</pose>
-      <visualize>$(arg laser_visual)</visualize>
-      <update_rate>5</update_rate>
+      <visualize>true</visualize>
+      <update_rate>40</update_rate>
       <ray>
         <scan>
           <horizontal>
-            <samples>360</samples>
+            <samples>1000</samples>
             <resolution>1</resolution>
-            <min_angle>0.0</min_angle>
-            <max_angle>6.28319</max_angle>
+            <min_angle>-2.3562</min_angle>
+            <max_angle>2.3562</max_angle>
           </horizontal>
         </scan>
         <range>
-          <min>0.120</min>
-          <max>3.5</max>
-          <resolution>0.015</resolution>
+          <min>0.06</min>
+          <max>4.0</max>
+          <resolution>0.001</resolution>
         </range>
         <noise>
           <type>gaussian</type>
           <mean>0.0</mean>
-          <stddev>0.01</stddev>
+          <stddev>0.03</stddev>
         </noise>
       </ray>
-      <plugin name="gazebo_ros_lds_lfcd_controller" filename="libgazebo_ros_laser.so">
+      <plugin name="urg_lrf_controller" filename="libgazebo_ros_laser.so">
         <topicName>scan</topicName>
         <frameName>base_scan</frameName>
@@ -73,9 +72,8 @@
     </sensor>
   </gazebo>
-<!--link : https://www.raspberrypi.org/documentation/hardware/camera/-->
   <gazebo reference="camera_rgb_frame">
     <sensor type="camera" name="Pi Camera">
       <always_on>true</always_on>
-      <visualize>$(arg camera_visual)</visualize>
+      <visualize>true</visualize>
       <camera>
           <horizontal_fov>1.085595</horizontal_fov>

Commit message: resize beego

File: potbot_description/urdf/beego2.urdf.xacro (robot description, xacro)
@@ -15,19 +15,19 @@
   <link name="base_link">
     <visual>
-      <origin xyz="-0.08 0 0.1"/>
-      <geometry>
-        <box size="0.2 0.2 0.2"/>
+      <origin xyz="-0.08 0 0.115"/>
+      <geometry>
+        <box size="0.2 0.2 0.23"/>
       </geometry>
       <material name="grey" />
     </visual>
     <collision>
-      <origin xyz="-0.08 0.1"/>
-      <geometry>
-        <box size="0.2 0.2 0.2"/>
-      </geometry>
-    </collision>
-    <inertial>
-      <origin xyz="0 0 0"/>
-      <xacro:box_inertial mass="5" height="0.2" width="0.2" depth="0.2"/>
+      <origin xyz="-0.08 0.115"/>
+      <geometry>
+        <box size="0.2 0.2 0.23"/>
+      </geometry>
+    </collision>
+    <inertial>
+      <origin xyz="0 0 0"/>
+      <xacro:box_inertial mass="5" height="0.2" width="0.2" depth="0.23"/>
     </inertial>
   </link>
@@ -109,5 +109,5 @@
     <parent link="base_link" />
     <child link="base_scan" />
-    <origin xyz="0.09 0 0.223" rpy="${M_PI} 0 0"/>
+    <origin xyz="0.1 0 0.18" rpy="${M_PI} 0 0"/>
   </joint>
   <link name="base_scan">
@@ -128,5 +128,5 @@
   </link>
   <joint name="camera_stay_joint" type="fixed">
-    <origin xyz="0.06 0 0.2275" rpy="0 0 0"/>
+    <origin xyz="0.065 0 0.26" rpy="0 0 0"/>
     <parent link="base_link"/>
     <child link="camera_stay_link"/>
@@ -136,5 +136,5 @@
       <origin xyz="0 0 0" rpy="0 0 0"/>
       <geometry>
-        <box size="0.02 0.02 0.455"/>
+        <box size="0.02 0.02 0.29"/>
       </geometry>
       <material name="grey" />
@@ -143,15 +143,15 @@
       <origin xyz="0 0 0" rpy="0 0 0"/>
       <geometry>
-        <box size="0.02 0.02 0.455"/>
-      </geometry>
-    </collision>
-    <inertial>
-      <origin xyz="0 0 0"/>
-      <xacro:box_inertial mass="0.5" height="0.455" width="0.02" depth="0.02"/>
+        <box size="0.02 0.02 0.29"/>
+      </geometry>
+    </collision>
+    <inertial>
+      <origin xyz="0 0 0"/>
+      <xacro:box_inertial mass="0.5" height="0.29" width="0.02" depth="0.02"/>
     </inertial>
   </link>
   <joint name="pan_joint" type="revolute">
     <axis xyz="0 0 1"/>
-    <origin xyz="0 0 0.2375" rpy="0 0 0"/>
+    <origin xyz="0.035 0 0.145" rpy="0 0 0"/>
     <limit lower="-0.87" upper="0.87" effort="100" velocity="100"/>
     <parent link="camera_stay_link"/>

Commit message: desktop

File: potbot_description/urdf/beego2.urdf.xacro (robot description, xacro)
@@ -22,5 +22,5 @@
     </visual>
     <collision>
-      <origin xyz="-0.08 0.115"/>
+      <origin xyz="-0.08 0 0.115"/>
       <geometry>
         <box size="0.2 0.2 0.23"/>

Commit message: ros-pc

File: potbot_description/urdf/beego2.urdf.xacro (robot description, xacro)
@@ -15,5 +15,5 @@
   <link name="base_link">
     <visual>
-      <origin xyz="-0.08 0 0.115"/>
+      <origin xyz="-0.08 0 0.115" rpy="0 0 0"/>
       <geometry>
         <box size="0.2 0.2 0.23"/>
@@ -22,5 +22,5 @@
     </visual>
     <collision>
-      <origin xyz="-0.08 0 0.115"/>
+      <origin xyz="-0.08 0 0.115" rpy="0 0 0"/>
       <geometry>
         <box size="0.2 0.2 0.23"/>

Commit message: robot_localization

File: potbot_description/urdf/beego2.urdf.xacro (robot description, xacro)
@@ -240,5 +240,5 @@
   <link name="left_camera_frame"/>
   <joint name="left_camera_optical_joint" type="fixed">
-    <origin xyz="0 0 0" rpy="-1.57 0 -1.57"/>
+    <origin xyz="0 0 0" rpy="${-M_PI/2} 0 ${-M_PI/2}"/>
     <parent link="left_camera_frame"/>
     <child link="left_camera_optical_frame"/>
@@ -252,5 +252,5 @@
   <link name="right_camera_frame"/>
   <joint name="right_camera_optical_joint" type="fixed">
-    <origin xyz="0 0 0" rpy="-1.57 0 -1.57"/>
+    <origin xyz="0 0 0" rpy="${-M_PI/2} 0 ${-M_PI/2}"/>
     <parent link="right_camera_frame"/>
     <child link="right_camera_optical_frame"/>

File: potbot_description/urdf/megarover21.gazebo.xacro (robot description, xacro)
@@ -4,4 +4,13 @@
   <xacro:arg name="camera_visual" default="false"/>
   <xacro:arg name="imu_visual"    default="false"/>
+  <!-- If tf_prefix is given, use "frame tf_prefix/imu_frame", else "imu_frame" -->
+  <xacro:arg name="tf_prefix" default="" />
+  <xacro:property name="tf_prefix" value="$(arg tf_prefix)" />
+  <xacro:if value="${tf_prefix == ''}">
+      <xacro:property name="imu_frame" value="imu_link" />
+  </xacro:if>
+  <xacro:unless value="${tf_prefix == ''}">
+      <xacro:property name="imu_frame" value="$(arg tf_prefix)/imu_link" />
+  </xacro:unless>
   <gazebo reference="base_link">
     <selfCollide>false</selfCollide>
@@ -75,7 +84,8 @@
     </sensor>
   </gazebo>
-  <gazebo>
+  <!-- <gazebo>
     <plugin name="imu_plugin" filename="libgazebo_ros_imu.so">
       <alwaysOn>true</alwaysOn>
+      <frameName>imu_link</frameName>
       <bodyName>imu_link</bodyName>
       <topicName>imu</topicName>
@@ -83,5 +93,28 @@
       <gaussianNoise>0.0</gaussianNoise>
       <updateRate>20.0</updateRate>
+      <xyzOffset>0 0 0</xyzOffset>
+      <rpyOffset>0 0 0</rpyOffset>
+      <initialOrientationAsReference>false</initialOrientationAsReference>
     </plugin>
+  </gazebo> -->
+  <gazebo reference="imu_link">
+    <!-- <gravity>true</gravity> -->
+    <sensor name="imu_sensor" type="imu">
+      <always_on>true</always_on>
+      <update_rate>100</update_rate>
+      <visualize>true</visualize>
+      <topic>imu</topic>
+      <plugin filename="libgazebo_ros_imu_sensor.so" name="imu_plugin">
+        <topicName>imu</topicName>
+        <bodyName>imu_link</bodyName>
+        <updateRateHZ>30.0</updateRateHZ>
+        <gaussianNoise>0.0</gaussianNoise>
+        <xyzOffset>0 0 0</xyzOffset>
+        <rpyOffset>0 0 0</rpyOffset>
+        <frameName>${imu_frame}</frameName>
+        <initialOrientationAsReference>false</initialOrientationAsReference>
+      </plugin>
+      <pose>0 0 0 0 0 0</pose>
+    </sensor>
   </gazebo>
   <gazebo reference="left_camera_frame">

File: potbot_description/urdf/megarover21.urdf.xacro (robot description, xacro)
@@ -150,5 +150,5 @@
     <parent link="camera_link"/>
     <child link="imu_link"/>
-    <origin xyz="0 0 0" rpy="0 0 0"/>
+    <origin xyz="0 0 0" rpy="3.14 0 0"/>
   </joint>
   <link name="imu_link"/>
@@ -160,5 +160,5 @@
   <link name="left_camera_frame"/>
   <joint name="left_camera_optical_joint" type="fixed">
-    <origin xyz="0 0 0" rpy="-1.57 0 -1.57"/>
+    <origin xyz="0 0 0" rpy="${-M_PI/2} 0 ${-M_PI/2}"/>
     <parent link="left_camera_frame"/>
     <child link="left_camera_optical_frame"/>
@@ -172,5 +172,5 @@
   <link name="right_camera_frame"/>
   <joint name="right_camera_optical_joint" type="fixed">
-    <origin xyz="0 0 0" rpy="-1.57 0 -1.57"/>
+    <origin xyz="0 0 0" rpy="${-M_PI/2} 0 ${-M_PI/2}"/>
     <parent link="right_camera_frame"/>
     <child link="right_camera_optical_frame"/>
