Commit message: actual

File: potbot_description/urdf/megarover21.urdf.xacro (robot description, xacro)
@@ -150,5 +150,6 @@
     <parent link="camera_link"/>
     <child link="imu_link"/>
-    <origin xyz="0 0 0" rpy="3.14 0 0"/>
+    <!-- <origin xyz="0 0 0" rpy="3.14 0 0"/> -->
+    <origin xyz="0 0 0" rpy="0 1.57 0"/>
   </joint>
   <link name="imu_link"/>
